File: USB 2.0 Hub.kicad_pcb (KiCad board)
At the start: 2 copper layers, 57.4 x 27.9 mm, 32 parts, among them J1 USB_C_Receptacle_USB2.0, J2 USB_C_Receptacle_USB2.0, J3 USB_C_Receptacle_USB2.0, J4 USB_C_Receptacle_USB2.0, J5 USB_C_Receptacle_USB2.0, U1 SL2.1A

Commit message: Add files via upload
Connections:
- R10 pad 2: GND -> /VBUS
- R3 pad 1: GND -> /VBUS
- R4 pad 2: GND -> /VBUS
- R5 pad 1: GND -> /VBUS
- R6 pad 2: GND -> /VBUS
- R7 pad 1: GND -> /VBUS
- R8 pad 2: GND -> /VBUS
- R9 pad 1: GND -> /VBUS
Routing:
- net /VBUS: track 162.8 -> 186.2 mm
