File: USB 2.0 Hub.kicad_sch (KiCad schematic)
At the start: 30 parts, among them J1 USB_C_Receptacle_USB2.0, J2 USB_C_Receptacle_USB2.0, J3 USB_C_Receptacle_USB2.0, J4 USB_C_Receptacle_USB2.0, J5 USB_C_Receptacle_USB2.0, U1 SL2.1A

Commit message: Add files via upload
Connections:
- net GND: no longer R10.2, R3.1, R4.2, R5.1, R6.2, R7.1, R8.2, R9.1
- net VBUS: now also R10.2, R3.1, R4.2, R5.1, R6.2, R7.1, R8.2, R9.1
